File: prototype/cpuboard/prototype.kicad_pcb (KiCad board)
At the start: 4 copper layers, 78.7 x 63.5 mm, 13 parts, among them P1 CONN_25X2, P2 CONN_25X2, U1 MC68SEC000

Commit message: PCB labels
Other:
- board text added: "68SEC000 CPU"
- board text added: "68k Computer Prototype"
- board text added: "CPU Board v0.1"
Changed lines of the file:
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@@
     (area 112.344999 60.909999 191.185001 124.510001)
     (thickness 1.6)
-    (drawings 8)
+    (drawings 13)
     (tracks 320)
     (zones 0)
@@
     (visible_elements 7FFFFFFF)
     (pcbplotparams
-      (layerselection 0x00000_00000001)
+      (layerselection 0x010f0_80000007)
       (usegerberextensions false)
-      (excludeedgelayer false)
+      (excludeedgelayer true)
       (linewidth 0.100000)
       (plotframeref false)
@@
       (padsonsilk true)
       (subtractmaskfromsilk false)
-      (outputformat 4)
+      (outputformat 1)
       (mirror false)
       (drillshape 0)
@@
     )
   )
+  (gr_text "68SEC000 CPU" (at 157.48 88.9 315) (layer F.SilkS)
+    (effects (font (size 0.762 0.762) (thickness 0.1905)))
+  )
+  (gr_text "CPU Board v0.1" (at 128.27 114.3) (layer B.SilkS)
+    (effects (font (size 1.5 1.5) (thickness 0.3)) (justify mirror))
+  )
+  (gr_text "68k Computer Prototype" (at 170.18 114.3) (layer B.SilkS)
+    (effects (font (size 1.5 1.5) (thickness 0.3)) (justify mirror))
+  )
+  (gr_text "CPU Board v0.1" (at 175.26 114.3) (layer F.SilkS)
+    (effects (font (size 1.5 1.5) (thickness 0.3)))
+  )
+  (gr_text "68k Computer Prototype" (at 133.35 114.3) (layer F.SilkS)
+    (effects (font (size 1.5 1.5) (thickness 0.3)))
+  )
   (gr_line (start 114.6175 124.46) (end 188.9125 124.46) (angle 90) (layer Edge.Cuts) (width 0.1))
